File: 65-xt.kicad_pcb (KiCad board)
At the start: 2 copper layers, 177 parts, among them J1 Conn_01x04, Q1 2N7002, SW1 SW_Push, U1 MCP1700-3302E_SOT23, U2 STM32F072CBT6

Commit message: remove submodule, update footprints
Parts:
- SW1: footprint acheron_Hardware:K2-1187SQ-A4SW-06 -> random-keyboard-parts:SKQG-1155865
Routing:
- net +3V3: track 131.4 -> 115.1 mm
- net BOOT0: track 80.8 -> 67.9 mm
Other:
- board outline added: 346.7 x 94.3 mm

Commit message: adjust reset switch position, add tear drops, add board art
Parts:
- added G***: LOGO, board_logos:i65-xt-silk, B.Cu at (289.7, 244.5)
- added G***: LOGO, board_logos:o-logo, F.Cu at (349.2, 244.5)
- SW1: footprint random-keyboard-parts:SKQG-1155865 -> footprints-and-logos:K2-1187SQ-A4SW-06
- moved D18 7.05 mm to (474.0, 171.7), turned to 0 degrees
- moved D51 7.05 mm to (474.0, 209.8), turned to 0 degrees
- moved D67 7.05 mm to (474.0, 228.9), turned to 0 degrees
- moved D77 7.05 mm to (474.0, 247.9), turned to 0 degrees
- moved D35 7.05 mm to (474.0, 190.8), turned to 0 degrees
- moved SW1 1.59 mm to (208.0, 206.4)
Routing:
- net +3V3: track 115.1 -> 134.6 mm
- net BOOT0: track 67.9 -> 82.2 mm
- net Row4: track 399.2 -> 390.7 mm
- net Row3: track 373.6 -> 365.1 mm
- net Row2: track 337.5 -> 329.0 mm
- net Row0: track 477.1 -> 468.6 mm
- net Row1: track 353.0 -> 344.5 mm
- net Net-(D51-Pad2): track 7.36 -> 8.51 mm
- net Net-(D67-Pad2): track 7.36 -> 8.51 mm
- net Net-(D18-Pad2): track 7.36 -> 8.51 mm
- net Net-(D77-Pad2): track 7.36 -> 8.51 mm
- net Net-(D35-Pad2): track 7.36 -> 8.51 mm
Other:
- outline, holes or cut-outs redrawn

Commit message: update edge cuts
Other:
- outline, holes or cut-outs redrawn
